Commit message: lab2 fin

File: src/testbot_lab2/urdf/first.urdf (robot description, URDF)
Before this commit: robot robot, 4 links, 3 joints
Links:
- link link2: geometry visual box size=${i3['link_len']} 0.002 0.002

File: src/testbot_lab2/urdf/second.urdf (robot description, URDF)
Before this commit: robot robot, 4 links, 3 joints
Links:
- link base_link: geometry visual cylinder length=0.04 radius=0.04
- link link3: geometry visual box size=0.04 0.04 0.2

Commit message: LAB2 FIN

File: src/testbot_lab2/urdf/first.urdf (robot description, URDF)
Before this commit: robot robot, 4 links, 3 joints
Links:
- link base_link: geometry visual cylinder length=0.04 radius=0.04
- link link2: geometry visual box size=${i3['link_len']} 0.04 0.04
- link link3: geometry visual box size=0.04 0.04 0.2
